File: hardware/dda/dda.sch (EAGLE design)
At the start: 63 parts, among them IC1 74LS132D, K1 CP1-12V, T1 BC847, T2 BC847, T3 BC847, T4 BC847, T5 BC847, T6 BC847, T7 BC847, T8 BC847, T9 BC847

Commit message: DDA board routed v1.0b
Parts:
- removed A_MOTOR, B_MOTOR, D_MOTOR, G_MOTOR: 22-23-2041, con-molex:22-23-2041
- removed D, G: STEPPER, stepper_module:STEPPER
- removed ENDSTOP_A, ENDSTOP_B, ENDSTOP_D, ENDSTOP_G: 22-23-2021, con-molex:22-23-2021
- added C10, C11: 18p, rcl:C-EUC0805
- added C12, C13: 2.2u, rcl:C-EUC1206
- added C14, C5, C6, C7, C8, C9: 100n, rcl:C-EUC0805
- added C15: 10u, rcl:CPOL-EUCT3216
- added C16, C17, C18, C19: 220u, Panasonic-EEEFT_EEEH:EEE-FTE221XAP-CASE-D8
- added D10: RED, led:LEDCHIP-LED0805
- added D11: BAT60JFILM, diode:BAT60J
- added H1, H2, H3, H4: MOUNT-HOLE3.2, holes:MOUNT-HOLE3.2
- added IC2: STM32F407VGT, micro-stm_v2:STM32F407VGT
- added IC3: LD1117, v-reg:LD117AS12TR
- added JP1, JP2, JP3: (no value), pinhead-2:PINHD-1X03_2.00
- added MOTOR_A, MOTOR_B, MOTOR_D, MOTOR_G, PWR: 22-23-2041, con-molex:22-23-2041
- added Q1: FDN304P, transistor-power:FDN360P
- added R28, R29, R30: 10K, rcl:R-EU_M0805
- added R31: 4K7, rcl:R-EU_M0805
- added R32, R36: 20K, rcl:R-EU_M0805
- added R33, R35: 0R, rcl:R-EU_R0805W
- added R34: 100R, rcl:R-EU_M0805
- added RAP: MICROMATCH-14, con-amp-micromatch:MICROMATCH-14
- added STEPPER_D, STEPPER_G: REPICO_STEPPER, stepper_module:REPICO_STEPPER
- added SWD: MICROMATCH-6, con-amp-micromatch:MICROMATCH-6
- added T10: BC847, transistor:BC847
- added X1, X2, X3, X4: 22-23-2021, con-molex:22-23-2021
- added Y1: 8MHz, Simplex-FreqCtrl:CRYSTAL5X3.2
- C1, C4: value 10u -> 100n; device rcl:C-EUC0805K -> rcl:C-EUC0805; FARNELL 2496944 -> (none); PARTNO (none) -> 2496944; PRICE 0.171 -> (none)
- C2, C3: device rcl:C-EUC0805K -> rcl:C-EUC0805; FARNELL 2496944 -> (none); PARTNO (none) -> 2496944; PRICE 0.171 -> (none)
- D1, D2, D3, D4: FARNELL 1466524 -> (none); PARTNO (none) -> 1466524; PRICE 0.0651 -> (none)
- D5, D6, D7, D8: value (none) -> YELLOW; FARNELL 1716768 -> (none); PARTNO (none) -> 1581241; PRICE 0.312 -> (none)
- D9: value (none) -> RED; FARNELL 1716765 -> (none); PARTNO (none) -> 1581239
- IC1: value 74LS132D -> CD74HC32M; FARNELL 1103158 -> (none); PARTNO (none) -> 1103158; PRICE 0.739 -> (none)
- K1: FARNELL 2103582 -> (none); PARTNO (none) -> 2103582; PRICE 2.84 -> (none)
- R1: value 3K3 -> 4K7; PARTNO (none) -> 9333266
- R10: value 330 -> 560R; PARTNO (none) -> 9334688
- R11, R13, R15, R16, R19, R20, R23, R24: value 470 -> 560R; PARTNO (none) -> 9334688
- R12, R17, R21, R25: value 12K -> 10K; PARTNO (none) -> 9332391
- R14, R18, R22, R26: PARTNO (none) -> 9333266
- R2, R3, R4, R5, R6, R7, R8, R9: FARNELL 1469911 -> (none); PARTNO (none) -> 9333045; PRICE 0.0157 -> (none)
- R27: value 3K3 -> 20K; PARTNO (none) -> 9332774
- STEPPER_A, STEPPER_B: value STEPPER -> REPICO_STEPPER; device stepper_module:STEPPER -> stepper_module:REPICO_STEPPER; PARTNO (none) -> 1593462
- T1, T2, T3, T4, T5, T6, T7, T8, T9: PARTNO (none) -> 2432696
Connections:
- removed net 12V_ENABLE: R1.1, R27.2
- removed net ENDSTOP_A: IC1B.O
- removed net ENDSTOP_B: IC1A.O
- removed net ENDSTOP_D: IC1C.O
- removed net ENDSTOP_G: IC1D.O
- removed net N$10: G.OUT1A, G_MOTOR-2.S
- removed net N$11: G.OUT2A, G_MOTOR-3.S
- removed net N$12: G.OUT2B, G_MOTOR-4.S
- removed net N$13: D.OUT1B, D_MOTOR-1.S
- removed net N$14: D.OUT1A, D_MOTOR-2.S
- removed net N$15: D.OUT2A, D_MOTOR-3.S
- removed net N$16: D.OUT2B, D_MOTOR-4.S
- removed net N$19: D1.A, ENDSTOP_A-1.S, R2.1, R3.1
- removed net N$21: D2.A, ENDSTOP_B-1.S, R4.1, R5.1
- removed net N$23: D3.A, ENDSTOP_G-1.S, R6.1, R7.1
- removed net N$25: D4.A, ENDSTOP_D-1.S, R8.1, R9.1
- removed net N$4: A_MOTOR-4.S, STEPPER_A.OUT2B
- removed net N$6: B_MOTOR-2.S, STEPPER_B.OUT1A
- removed net N$7: B_MOTOR-3.S, STEPPER_B.OUT2A
- removed net N$8: B_MOTOR-4.S, STEPPER_B.OUT2B
- new net 12V_ENBL: IC2MCU.PC0, R1.1, R27.2
- new net 3_3V_ENBL: JP2.2, R31.2
- new net A_ENDST: IC1B.O, IC2MCU.PC4
- new net A_ENDSW: D1.A, R2.1, R3.1, X1-1.S
- new net A_OUT1A: MOTOR_A-2.S, STEPPER_A.OUT1A
- new net A_OUT1B: MOTOR_A-1.S, STEPPER_A.OUT1B
- new net A_OUT2A: MOTOR_A-3.S, STEPPER_A.OUT2A
- new net A_OUT2B: MOTOR_A-4.S, STEPPER_A.OUT2B
- new net BOOT1: IC2MCU.PB2, R28.2
- new net B_ENDST: IC1A.O, IC2MCU.PC5
- new net B_ENDSW: D2.A, R4.1, R5.1, X2-1.S
- new net B_OUT1A: MOTOR_B-2.S, STEPPER_B.OUT1A
- new net B_OUT1B: MOTOR_B-1.S, STEPPER_B.OUT1B
- new net B_OUT2A: MOTOR_B-3.S, STEPPER_B.OUT2A
- new net B_OUT2B: MOTOR_B-4.S, STEPPER_B.OUT2B
- new net D_ENDST: IC1C.O, IC2MCU.PC14
- new net D_ENDSW: D4.A, R8.1, R9.1, X4-1.S
- new net D_OUT1A: MOTOR_D-2.S, STEPPER_D.OUT1A
- new net D_OUT1B: MOTOR_D-1.S, STEPPER_D.OUT1B
- new net D_OUT2A: MOTOR_D-3.S, STEPPER_D.OUT2A
- new net D_OUT2B: MOTOR_D-4.S, STEPPER_D.OUT2B
- new net EXT_3_3V: JP3.3, R33.2, R35.2
- new net G_ENDST: IC1D.O, IC2MCU.PC13
- new net G_ENDSW: D3.A, R6.1, R7.1, X3-1.S
- new net G_OUT1A: MOTOR_G-2.S, STEPPER_G.OUT1A
- new net G_OUT1B: MOTOR_G-1.S, STEPPER_G.OUT1B
- new net G_OUT2A: MOTOR_G-3.S, STEPPER_G.OUT2A
- new net G_OUT2B: MOTOR_G-4.S, STEPPER_G.OUT2B
- new net NRST: IC2MCU.NRST, JP1.2
- new net OSC_IN: C10.2, IC2MCU.OSC_IN, Y1.2
- new net OSC_OUT: C11.2, IC2MCU.OSC_OUT, Y1.1
- new net RAP_3_3V: JP3.1, RAP-1.S, RAP-2.S
- new net RAP_BOOTSEL: IC2MCU.BOOT0, R29.1, RAP-9.S
- new net RAP_ENBL: JP2.1, RAP-3.S
- new net RAP_INT0: IC2MCU.PC1, RAP-10.S
- new net RAP_INT1: IC2MCU.PD3, RAP-11.S
- new net RAP_INT2: IC2MCU.PD4, RAP-12.S
- new net RAP_NRST: JP1.1, RAP-4.S
- new net SPI_MISO: IC2MCU.PC2, RAP-8.S
- new net SPI_MOSI: IC2MCU.PC3, RAP-7.S
- new net SPI_NSS: IC2MCU.PB12, RAP-5.S
- new net SPI_SCK: IC2MCU.PB10, RAP-6.S
- new net SUPPLY_3_3V: JP2.3, JP3.2, Q1.S, R30.2
- new net SUPPLY_5V: C14.1, IC3.IN, PWR-2.S
- new net SWCLK: IC2MCU.PA14, SWD-2.S
- new net SWDIO: IC2MCU.PA13, SWD-3.S
- new net SWD_NRST: JP1.3, SWD-4.S
- new net SWO: IC2MCU.PB3, SWD-5.S
- new net VCAP_1: C12.1, IC2MCU.VCAP2
- new net VCAP_2: C13.1, IC2MCU.VCAP1
- net 12V: now also C16.1, C17.1, C18.1, C19.1, STEPPER_D.VCC, STEPPER_G.VCC; no longer D.VCC, G.VCC
- net 3_3V: now also C5.1, C6.1, C7.1, C8.1, C9.1, IC2MCU.VDDA, IC2MCU.VREF+, IC2PWR.VDD@1, IC2PWR.VDD@2, IC2PWR.VDD@3, IC2PWR.VDD@4, IC2PWR.VDD@5, IC2PWR.VDD@6, Q1.D, R29.2, R32.2, R34.2, STEPPER_D.VDD, STEPPER_G.VDD; no longer D.VDD, G.VDD
- net A_DIR: now also IC2MCU.PD8
- net A_DIS: now also IC2MCU.PD5
- net A_MS1: now also IC2MCU.PD7
- net A_MS2: now also IC2MCU.PD6
- net A_STEP: now also IC2MCU.PD9
- net B_DIR: now also IC2MCU.PC7
- net B_DIS: now also IC2MCU.PC6
- net B_MS1: now also IC2MCU.PD10
- net B_MS2: now also IC2MCU.PD11
- net B_STEP: now also IC2MCU.PC8
- net D_DIR: now also IC2MCU.PD13, STEPPER_D.DIR; no longer D.DIR
- net D_DIS: now also IC2MCU.PD12, STEPPER_D.DIS; no longer D.DIS
- net D_MS1: now also IC2MCU.PD1, STEPPER_D.MS1; no longer D.MS1
- net D_MS2: now also IC2MCU.PD2, STEPPER_D.MS2; no longer D.MS2
- net D_STEP: now also IC2MCU.PD14, STEPPER_D.STEP; no longer D.STEP
- net GND: now also C10.1, C11.1, C12.2, C13.2, C14.2, C15.-, C16.2, C17.2, C18.2, C19.2, C5.2, C6.2, C7.2, C8.2, C9.2, D10.C, IC2MCU.VSSA, IC2PWR.VSS@1, IC2PWR.VSS@2, IC2PWR.VSS@3, IC2PWR.VSS@4, IC3.ADJ, PWR-3.S, PWR-4.S, R28.1, R32.1, R36.1, RAP-13.S, RAP-14.S, STEPPER_D.GND, STEPPER_G.GND, SWD-6.S, T10.E, X1-2.S, X2-2.S, X3-2.S, X4-2.S; no longer D.GND, ENDSTOP_A-2.S, ENDSTOP_B-2.S, ENDSTOP_D-2.S, ENDSTOP_G-2.S, G.GND
- net G_DIR: now also IC2MCU.PC15, STEPPER_G.DIR; no longer G.DIR
- net G_DIS: now also IC2MCU.PC12, STEPPER_G.DIS; no longer G.DIS
- net G_MS1: now also IC2MCU.PC10, STEPPER_G.MS1; no longer G.MS1
- net G_MS2: now also IC2MCU.PC11, STEPPER_G.MS2; no longer G.MS2
- net G_STEP: now also IC2MCU.PD0, STEPPER_G.STEP; no longer G.STEP
- net N$1: now also Q1.G, R30.1, T10.C; no longer A_MOTOR-1.S, STEPPER_A.OUT1B
- net N$17: now also D11.A
- net N$2: now also R35.1, SWD-1.S; no longer A_MOTOR-2.S, STEPPER_A.OUT1A
- net N$3: now also R31.1, R36.2, T10.B; no longer A_MOTOR-3.S, STEPPER_A.OUT2A
- net N$5: now also D10.A, R34.1; no longer B_MOTOR-1.S, STEPPER_B.OUT1B
- net N$9: now also C15.+, IC3.OUT, R33.1; no longer G.OUT1B, G_MOTOR-1.S
- net SUPPLY_12V: now also D11.C, PWR-1.S
Other:
- note added: "Connectors"
- note added: "Decoupling"
- note added: "Eventually use a BAT60JFILM for isolation"
- note added: "MCU"
- note added: "Power"
- note added: "Status LEDS"
